Commit message: Here I have completed both xacro file and gmapping.

File: urdf/mr_CCMDX1.urdf (robot description, URDF)
Before this commit: robot mr_CCMDX1, 13 links, 12 joints
Links:
- removed link camera
- removed link head
- added link camera_link, mass 1; collision box size=0.08 0.08 0.08; visual box size=0.08 0.08 0.08
- added link hokuyo_link, mass 1e-5; collision box size=0.1 0.1 0.1; visual mesh filename=package://mobile_robot_CCMDX1/meshes/hokuyo.dae
- added link robot_head_link, mass 5; collision sphere radius=0.2; visual sphere radius=0.2
Joints:
- removed joint tobox
- added joint camera_box_joint: type fixed, parent robot_head_link, child camera_link, origin xyz=0.1814 0 0.1414, axis 0 1 0
- added joint head_laser_sensor_joint: type fixed, parent robot_head_link, child hokuyo_link, origin xyz=0 0 0.23, axis 0 0 0
- joint head_swivel_joint: child head -> robot_head_link
