Commit message: this version is after I worked on SLAM

File: urdf/01_mr_CCMDX1.urdf.xacro (robot description, xacro)
@@ -1,4 +1,5 @@
 <?xml version="1.0"?>
 <robot name="mr_CCMDX1" xmlns:xacro="http://ros.org/wiki/xacro">
+<origin xyz="0 0 1"/>
   <xacro:property name="width" value="0.2" />
   <xacro:property name="wheelradius" value="0.05" />
@@ -72,12 +73,56 @@
   <transmission name="head_swivel_trans">
     <type>transmission_interface/SimpleTransmission</type>
+    <joint name="head_swivel_joint">
+      <!--hardwareInterface>hardware_interface/PositionJointInterface</hardwareInterface-->
+      <hardwareInterface>hardware_interface/PositionJointInterface</hardwareInterface>
+    </joint>
     <actuator name="$head_swivel_motor">
       <mechanicalReduction>1</mechanicalReduction>
+      <hardwareInterface>hardware_interface/PositionJointInterface</hardwareInterface>
     </actuator>
-    <joint name="head_swivel_joint">
-      <!--hardwareInterface>hardware_interface/PositionJointInterface</hardwareInterface-->
-	<hardwareInterface>hardware_interface/PositionJointInterface</hardwareInterface>
-    </joint>
   </transmission>
+<!-- Here I need to add the stabiliser macro -->
+ <xacro:macro name="stabiliser" params="suffix_s reflect_s"> <!-- this macro will accept two parameters: suffix and reflect-->
+   <link name="${suffix_s}_stabiliser_link">
+    <visual>
+     <geometry>
+      <sphere radius="${width/3}"/>
+     </geometry>
+     <origin xyz="0 0 0" rpy="0 0 0"/>
+     <material name="black"/>
+    </visual>
+    <collision>
+     <geometry>
+      <sphere radius="${width/3}"/>
+     </geometry>
+     <origin xyz="0 0 0" rpy="0 0 0"/>
+    </collision>
+    <xacro:mdxcc1_inertial mass="4"/>
+   </link>
+   <joint name="${suffix_s}_stabiliser_joint" type="continuous">
+    <parent link="base_link"/>
+    <child link="${suffix_s}_stabiliser_link"/>
+    <axis xyz="0 0 1"/>
+    <origin xyz="${reflect_s*(0.07+(width/2))} 0 -${0.03+width/2}"/>
+    <limit effort="50" velocity="0.5"/>
+  </joint>
+   <gazebo reference="${suffix_s}_stabiliser_link">
+    <mu1 value="200.0"/>
+    <mu2 value="100.0"/>
+    <kp value="10000000.0" />
+    <kd value="1.0" />
+    <material>Gazebo/Black</material>
+   </gazebo>
+    <transmission name="${suffix_s}_stabiliser_trans">
+      <type>transmission_interface/SimpleTransmission</type>
+      <joint name="${suffix_s}_stabiliser_joint">
+        <hardwareInterface>hardware_interface/VelocityJointInterface</hardwareInterface>
+      </joint>
+      <actuator name="${suffix_s}_stabiliser_motor">
+        <mechanicalReduction>1</mechanicalReduction>
+        <hardwareInterface>hardware_interface/VelocityJointInterface</hardwareInterface>
+      </actuator>
+    </transmission>
+ </xacro:macro>
 <!-- Here I need to add the wheel macro -->
   <xacro:macro name="wheel" params="prefix suffix reflect_w"> <!-- this macro will accept three parameters: prefix, suffix and reflect-->
@@ -113,10 +158,11 @@
     <transmission name="${prefix}_${suffix}_wheel_trans">
       <type>transmission_interface/SimpleTransmission</type>
-      <actuator name="${prefix}_${suffix}_wheel_motor">
-        <mechanicalReduction>1</mechanicalReduction>
-      </actuator>
       <joint name="${prefix}_${suffix}_wheel_joint">
         <hardwareInterface>hardware_interface/VelocityJointInterface</hardwareInterface>
       </joint>
+      <actuator name="${prefix}_${suffix}_wheel_motor">
+        <mechanicalReduction>1</mechanicalReduction>
+        <hardwareInterface>hardware_interface/VelocityJointInterface</hardwareInterface>
+      </actuator>
     </transmission>
   </xacro:macro>
@@ -200,4 +246,6 @@
   <xacro:leg prefix="right" reflect="-1" />
   <xacro:leg prefix="left" reflect="1" />
+  <xacro:stabiliser suffix_s="front" reflect_s="1" />
+  <xacro:stabiliser suffix_s="back" reflect_s="-1" />
   <joint name="camera_box_joint" type="fixed">
    <axis xyz="0 1 0" />
@@ -226,5 +274,5 @@
   </link>
     <gazebo reference="camera_link">
-      <material>Gazebo/White</material>
+      <material>Gazebo/YellowGlow</material>
     </gazebo>
 <!-- camera -->
@@ -271,6 +319,6 @@
  <joint name="head_laser_sensor_joint" type="fixed">
     <axis xyz="0 0 0" />
-    <origin xyz="0 0 0.30"/>
-    <parent link="robot_head_link"/>
+    <origin xyz="0 0 0.36"/>
+    <parent link="base_link"/>
     <child link="hokuyo_link"/>
   </joint>
@@ -278,5 +326,5 @@
    <origin xyz="0 0 0" rpy="0 0 0"/>
     <collision>
-      <origin xyz="0 0 -0.02" rpy="0 0 0"/>
+      <origin xyz="0 0 0" rpy="0 0 0"/>
       <geometry>
        <box size="0.05 0.05 0.05"/>
@@ -293,10 +341,10 @@
   </link>
     <gazebo reference="hokuyo_link">
-      <material>Gazebo/White</material>
+      <material>Gazebo/YellowGlow</material>
     </gazebo>
 <!-- hokuyo -->
   <gazebo reference="hokuyo_link">
     <sensor type="gpu_ray" name="head_hokuyo_sensor">
-      <pose>0 0 0.23 0 0 0</pose>
+      <pose>0 0 0 0 0 0</pose>
       <visualize>false</visualize>
       <update_rate>40</update_rate>
@@ -326,5 +374,5 @@
       </ray>
       <plugin name="gazebo_ros_head_hokuyo_controller" filename="libgazebo_ros_gpu_laser.so">
-        <topicName>/r2d2_diff_drive_controller/laser/scan</topicName>
+        <topicName>/ccmdx1/laser/scan</topicName>
         <frameName>hokuyo_link</frameName>
       </plugin>

Commit message: Finally both map and Odometry work

File: urdf/01_mr_CCMDX1.urdf.xacro (robot description, xacro)
@@ -87,16 +87,16 @@
     <visual>
      <geometry>
-      <sphere radius="${width/3}"/>
+      <cylinder radius="${wheelradius*2}" length= "${wheelwidth*3}"/>
      </geometry>
-     <origin xyz="0 0 0" rpy="0 0 0"/>
+     <origin xyz="0 0 0" rpy="${pi/2} 0 0"/>
      <material name="black"/>
     </visual>
     <collision>
      <geometry>
-      <sphere radius="${width/3}"/>
+      <cylinder radius="${wheelradius*2}" length= "${wheelwidth*3}"/>
      </geometry>
-     <origin xyz="0 0 0" rpy="0 0 0"/>
+     <origin xyz="0 0 0" rpy="${pi/2} 0 0"/>
     </collision>
-    <xacro:mdxcc1_inertial mass="4"/>
+    <xacro:mdxcc1_inertial mass="5"/>
    </link>
    <joint name="${suffix_s}_stabiliser_joint" type="continuous">
@@ -104,12 +104,12 @@
     <child link="${suffix_s}_stabiliser_link"/>
     <axis xyz="0 0 1"/>
-    <origin xyz="${reflect_s*(0.07+(width/2))} 0 -${0.03+width/2}"/>
+    <origin xyz="${reflect_s*(0.15+(width*0.3))} 0 -${0.01+width/2}"/>
     <limit effort="50" velocity="0.5"/>
   </joint>
    <gazebo reference="${suffix_s}_stabiliser_link">
-    <mu1 value="200.0"/>
-    <mu2 value="100.0"/>
-    <kp value="10000000.0" />
-    <kd value="1.0" />
+    <mu1 value="100"/>
+    <mu2 value="100"/>
+    <kp value="100000" />
+    <kd value="1" />
     <material>Gazebo/Black</material>
    </gazebo>
@@ -348,17 +348,17 @@
       <pose>0 0 0 0 0 0</pose>
       <visualize>false</visualize>
-      <update_rate>40</update_rate>
+      <update_rate>1000</update_rate>
       <ray>
         <scan>
           <horizontal>
-            <samples>720</samples>
+            <samples>1500</samples>
             <resolution>1</resolution>
-            <min_angle>-1.570796</min_angle>
-            <max_angle>1.570796</max_angle>
+            <min_angle>-3.1415</min_angle>
+            <max_angle>3.1415</max_angle>
           </horizontal>
         </scan>
         <range>
-          <min>0.10</min>
-          <max>30.0</max>
+          <min>0.22</min>
+          <max>35.0</max>
           <resolution>0.01</resolution>
         </range>
